Commit message: Update robot_core.xacro

File: robot_core.xacro (robot description, xacro)
@@ -1,4 +1,5 @@
 <?xml version="1.0"?>
 <robot xmlns:xacro="http://www.ros.org/wiki/xacro" >
+<xacro:include filename="inertial_macros.xacro" />
     <material name="white">
         <color rgba="1 1 1 1" />
@@ -13,37 +14,9 @@
         <color rgba="0 0 0 1"/>
     </material>
- <material name="red">
-     <color rgba="1 0 0 1"/>
- </material>
-    <!-- BASE LINK -->
+    <material name="red">
+        <color rgba="1 0 0 1"/>
+    </material>
     <link name="base_link">
     </link>
-    <joint name="chassis_joint" type="fixed">
-        <parent link="base_link"/>
-        <child link="chassis"/>
-        <origin xyz="-0.1 0 0"/>
-    </joint>
-    <link name="chassis">
-        <visual>
-            <origin xyz="0.15 0 0.075" rpy="0 0 0"/>
-            <geometry>
-                <box size="0.3 0.3 0.15"/>
-            </geometry>
-            <material name="white"/>
-        </visual>
-        <collision>
-            <origin xyz="0.15 0 0.075" rpy="0 0 0"/>
-            <geometry>
-                <box size="0.3 0.3 0.15"/>
-            </geometry>
-        </collision>
-        <xacro:inertial_box mass="0.5" x="0.3" y="0.3" z="0.15">
-            <origin xyz="0.15 0 0.075" rpy="0 0 0"/>
-        </xacro:inertial_box>
-    </link>
-    <gazebo reference="chassis">
-        <material>Gazebo/White</material>
-    </gazebo>
-    <!-- BASE_FOOTPRINT LINK -->
     <joint name="base_footprint_joint" type="fixed">
         <parent link="base_link"/>
@@ -53,82 +26,231 @@
     <link name="base_footprint">
     </link>
-    <!-- LEFT WHEEL -->
-    <joint name="left_wheel_joint" type="continuous">
-        <parent link="base_link"/>
-        <child link="left_wheel"/>
-        <origin xyz="0 0.175 0" rpy="-${pi/2} 0 0"/>
+    <joint name="body_joint" type="fixed">
+        <parent link="base_footprint"/>
+        <child link="body"/>
+        <origin xyz="0 0 0" rpy="0 0 0"/>
+    </joint>
+    <!-- ฐานหุ่นยนต์ -->
+    <link name="body">
+        <visual>
+            <geometry>
+                <mesh filename="file:///home/preeyanan/miniproject/meshes/body.dae" scale="1 1 1"/>
+            </geometry>
+        </visual>
+        <collision>
+            <geometry>
+                <mesh filename="file:///home/preeyanan/miniproject/meshes/body.dae" scale="1 1 1"/>
+            </geometry>
+        </collision>
+        <xacro:inertial_box mass="5" x="0.46" y="0.55" z="0.40">
+            <origin xyz="0 0 0" rpy="0 0 0"/>
+        </xacro:inertial_box>
+    </link>
+    <gazebo reference="body">
+        <material>Gazebo/White</material>
+    </gazebo>
+    <!-- === ล้อหน้า ซ้าย === -->
+    <joint name="front_right_wheel_joint" type="continuous">
+        <parent link="body"/>
+        <child link="front_right_wheel"/>
+        <origin xyz="-1 -0.5 0" rpy="${pi/2} 0 0"/>
+        <axis xyz="1 0 0"/>
+    </joint>
+    <link name="front_left_wheel">
+        <visual>
+            <geometry>
+                <mesh filename="file:///home/preeyanan/miniproject/meshes/frontwheel.dae" scale="1 1 1"/>
+            </geometry>
+        </visual>
+        <collision>
+            <geometry>
+                <mesh filename="file:///home/preeyanan/miniproject/meshes/frontwheel.dae" scale="1 1 1"/>
+            </geometry>
+        </collision>
+        <xacro:inertial_cylinder mass="0.6" length="0.1" radius="0.09">
+            <origin xyz="0 0 0" rpy="0 0 0"/>
+        </xacro:inertial_cylinder>
+    </link>
+    <gazebo reference="front_left_wheel">
+        <material>Gazebo/White</material>
+    </gazebo>
+    <!-- === ล้อหน้า ขวา === -->
+    <joint name="front_left_wheel_joint" type="continuous">
+        <parent link="body"/>
+        <child link="front_left_wheel"/>
+        <origin xyz="1 0.175 0" rpy="${pi/2} 0 0"/>
+        <axis xyz="-1 -1 0"/>
+    </joint>
+    <link name="front_right_wheel">
+        <visual>
+            <geometry>
+                <mesh filename="file:///home/preeyanan/miniproject/meshes/frontwheel.dae" scale="1 1 1"/>
+            </geometry>
+        </visual>
+        <collision>
+            <geometry>
+                <mesh filename="file:///home/preeyanan/miniproject/meshes/frontwheel.dae" scale="1 1 1"/>
+            </geometry>
+        </collision>
+        <xacro:inertial_cylinder mass="0.6" length="0.1" radius="0.09">
+            <origin xyz="0 0 0" rpy="0 0 0"/>
+        </xacro:inertial_cylinder>
+    </link>
+    <gazebo reference="front_right_wheel">
+        <material>Gazebo/White</material>
+    </gazebo>
+    <!-- === ล้อหลัง ซ้าย === -->
+    <joint name="back_left_wheel_joint" type="continuous">
+        <parent link="body"/>
+        <child link="back_left_wheel"/>
+        <origin xyz="-0.5 1 0" rpy="${pi/2} 0 0"/>
+        <axis xyz="1 0 0"/>
+    </joint>
+    <link name="back_left_wheel">
+        <visual>
+            <geometry>
+                <mesh filename="file:///home/preeyanan/miniproject/meshes/backwheel.dae" scale="1 1 1"/>
+            </geometry>
+        </visual>
+        <collision>
+            <geometry>
+                <mesh filename="file:///home/preeyanan/miniproject/meshes/backwheel.dae" scale="1 1 1"/>
+            </geometry>
+        </collision>
+        <xacro:inertial_cylinder mass="1" length="0.1" radius="0.12">
+            <origin xyz="0 0 0" rpy="0 0 0"/>
+        </xacro:inertial_cylinder>
+    </link>
+    <gazebo reference="back_left_wheel">
+        <material>Gazebo/White</material>
+    </gazebo>
+    <!-- === ล้อหลัง ขวา === -->
+    <joint name="back_right_wheel_joint" type="continuous">
+        <parent link="body"/>
+        <child link="back_right_wheel"/>
+        <origin xyz="-1 1 0" rpy="${pi/2} 0 0"/>
+        <axis xyz="1 0 0"/>
+    </joint>
+    <link name="back_right_wheel">
+        <visual>
+            <geometry>
+                <mesh filename="file:///home/preeyanan/miniproject/meshes/backwheel.dae" scale="1 1 1"/>
+            </geometry>
+        </visual>
+        <collision>
+            <geometry>
+                <mesh filename="file:///home/preeyanan/miniproject/meshes/backwheel.dae" scale="1 1 1"/>
+            </geometry>
+        </collision>
+        <xacro:inertial_cylinder mass="1" length="0.1" radius="0.12">
+            <origin xyz="0 0 0" rpy="0 0 0"/>
+        </xacro:inertial_cylinder>
+    </link>
+    <gazebo reference="back_right_wheel">
+        <material>Gazebo/White</material>
+    </gazebo>
+    <!-- === LR L === -->
+    <joint name="LR_L_joint" type="prismatic">
+        <parent link="body"/>
+        <child link="LR_L"/>
+        <origin xyz="0 1 0" rpy="0 0 0"/>
+        <axis xyz="1 0 0"/>
+        <limit lower="-1" upper="1" effort="1" velocity="1"/>
+    </joint>
+    <link name="LR_L">
+        <visual>
+            <geometry>
+                <mesh filename="file:///home/preeyanan/miniproject/meshes/LR.dae" scale="1 1 1"/>
+            </geometry>
+        </visual>
+        <collision>
+            <geometry>
+                <mesh filename="file:///home/preeyanan/miniproject/meshes/LR.dae" scale="1 1 1"/>
+            </geometry>
+        </collision>
+        <xacro:inertial_box mass="0.3" x="0.03" y="0.03" z="0.2">
+            <origin xyz="0 0 0" rpy="0 0 0"/>
+        </xacro:inertial_box>
+    </link>
+    <gazebo reference="LR_L">
+        <material>Gazebo/White</material>
+    </gazebo>
+    <!-- === LR R === -->
+    <joint name="LR_R_joint" type="prismatic">
+        <parent link="body"/>
+        <child link="LR_R"/>
+        <origin xyz="-0.066 -0.296 0.095" rpy="0 0 0"/>
+        <axis xyz="1 0 0"/>
+        <limit lower="-1" upper="1" effort="1" velocity="1"/>
+    </joint>
+    <link name="LR_R">
+        <visual>
+            <geometry>
+                <mesh filename="file:///home/preeyanan/miniproject/meshes/LR.dae" scale="1 1 1"/>
+            </geometry>
+        </visual>
+        <collision>
+            <geometry>
+                <mesh filename="file:///home/preeyanan/miniproject/meshes/LR.dae" scale="1 1 1"/>
+            </geometry>
+        </collision>
+        <xacro:inertial_box mass="0.3" x="0.03" y="0.03" z="0.2">
+            <origin xyz="0 0 0" rpy="0 0 0"/>
+        </xacro:inertial_box>
+    </link>
+    <gazebo reference="LR_R">
+        <material>Gazebo/White</material>
+    </gazebo>
+    <!-- === UD L === -->
+    <joint name="UD_L_joint" type="prismatic">
+        <parent link="LR_L"/>
+        <child link="UD_L"/>
+        <origin xyz="0 1.5 0" rpy="0 0 0"/>
         <axis xyz="0 0 1"/>
-    </joint>
-    <link name="left_wheel">
-        <visual>
-            <geometry>
-                <cylinder length="0.04" radius="0.05" />
-            </geometry>
-            <material name="orange"/>
-        </visual>
-        <collision>
-            <geometry>
-                <cylinder length="0.04" radius="0.05" />
-            </geometry>
-        </collision>
-        <xacro:inertial_cylinder mass="0.1" length="0.05" radius="0.05">
-            <origin xyz="0 0 0" rpy="0 0 0"/>
-        </xacro:inertial_cylinder>
-    </link>
-    <gazebo reference="left_wheel">
-        <material>Gazebo/Orange</material>
-    </gazebo>
-    <!-- RIGHT WHEEL -->
-    <joint name="right_wheel_joint" type="continuous">
-        <parent link="base_link"/>
-        <child link="right_wheel"/>
-        <origin xyz="0 -0.175 0" rpy="${pi/2} 0 0"/>
-        <axis xyz="0 0 -1"/>
-    </joint>
-    <link name="right_wheel">
-        <visual>
-            <geometry>
-                <cylinder length="0.04" radius="0.05" />
-            </geometry>
-            <material name="red"/>
-        </visual>
-        <collision>
-            <geometry>
-                <cylinder length="0.04" radius="0.05" />
-            </geometry>
-        </collision>
-        <xacro:inertial_cylinder mass="0.1" length="0.05" radius="0.05">
-            <origin xyz="0 0 0" rpy="0 0 0"/>
-        </xacro:inertial_cylinder>
-    </link>
-    <gazebo reference="right_wheel">
-        <material>Gazebo/Red</material>
-    </gazebo>
-    <!-- CASTER WHEEL -->
-    <joint name="caster_wheel_joint" type="fixed">
-        <parent link="chassis"/>
-        <child link="caster_wheel"/>
-        <origin xyz="0.24 0 0" rpy="0 0 0"/>
-    </joint>
-    <link name="caster_wheel">
-        <visual>
-            <geometry>
-                <sphere radius="0.05" />
-            </geometry>
-            <material name="black"/>
-        </visual>
-        <collision>
-            <geometry>
-                <sphere radius="0.05" />
-            </geometry>
-        </collision>
-        <xacro:inertial_sphere mass="0.1" radius="0.05">
-            <origin xyz="0 0 0" rpy="0 0 0"/>
-        </xacro:inertial_sphere>
-    </link>
-    <gazebo reference="caster_wheel">
-        <material>Gazebo/Black</material>
-        <mu1 value="0.0"/>
-        <mu2 value="0.0"/>
-    </gazebo>
+        <limit lower="-1" upper="1" effort="1" velocity="1"/>
+    </joint>
+    <link name="UD_L">
+        <visual>
+            <geometry>
+                <mesh filename="file:///home/preeyanan/miniproject/meshes/UDL.dae" scale="1 1 1"/>
+            </geometry>
+        </visual>
+        <collision>
+            <geometry>
+                <mesh filename="file:///home/preeyanan/miniproject/meshes/UDL.dae" scale="1 1 1"/>
+            </geometry>
+        </collision>
+        <xacro:inertial_box mass="0.2" x="0.03" y="0.03" z="0.15">
+            <origin xyz="0 0 0" rpy="0 0 0"/>
+        </xacro:inertial_box>
+    </link>
+    <gazebo reference="UD_L">
+        <material>Gazebo/White</material>
+    </gazebo>
+    <!-- === UD R === -->
+    <joint name="UD_R_joint" type="prismatic">
+        <parent link="LR_R"/>
+        <child link="UD_R"/>
+        <origin xyz="0 1 0" rpy="0 0 0"/>
+        <axis xyz="0 0 1"/>
+        <limit lower="-1" upper="1" effort="1" velocity="1"/>
+    </joint>
+    <link name="UD_R">
+        <visual>
+            <geometry>
+                <mesh filename="file:///home/preeyanan/miniproject/meshes/UDR.dae" scale="1 1 1"/>
+            </geometry>
+        </visual>
+        <collision>
+            <geometry>
+                <mesh filename="file:///home/preeyanan/miniproject/meshes/UDR.dae" scale="1 1 1"/>
+            </geometry>
+        </collision>
+        <xacro:inertial_box mass="0.2" x="0.03" y="0.03" z="0.15">
+            <origin xyz="0 0 0" rpy="0 0 0"/>
+        </xacro:inertial_box>
+    </link>
+    <gazebo reference="UD_R">
+        <material>Gazebo/White</material>
+   </gazebo>
 </robot>

Commit message: Update robot_core.xacro

File: robot_core.xacro (robot description, xacro)
@@ -35,10 +35,10 @@
         <visual>
             <geometry>
-                <mesh filename="file:///home/preeyanan/miniproject/meshes/body.dae" scale="1 1 1"/>
-            </geometry>
-        </visual>
-        <collision>
-            <geometry>
-                <mesh filename="file:///home/preeyanan/miniproject/meshes/body.dae" scale="1 1 1"/>
+                <mesh filename="file:///home/preeyanan/robotic2/src/articubot_nuy/meshes/body.dae" scale="1 1 1"/>
+            </geometry>
+        </visual>
+        <collision>
+            <geometry>
+                <mesh filename="file:///home/preeyanan/robotic2/src/articubot_nuy/meshes/body.dae" scale="1 1 1"/>
             </geometry>
         </collision>
@@ -54,5 +54,5 @@
         <parent link="body"/>
         <child link="front_right_wheel"/>
-        <origin xyz="-1 -0.5 0" rpy="${pi/2} 0 0"/>
+        <origin xyz="0.193 -0.1481 0.0198" rpy="${pi/2} 0 0"/>
         <axis xyz="1 0 0"/>
     </joint>
@@ -60,10 +60,10 @@
         <visual>
             <geometry>
-                <mesh filename="file:///home/preeyanan/miniproject/meshes/frontwheel.dae" scale="1 1 1"/>
-            </geometry>
-        </visual>
-        <collision>
-            <geometry>
-                <mesh filename="file:///home/preeyanan/miniproject/meshes/frontwheel.dae" scale="1 1 1"/>
+                <mesh filename="file:///home/preeyanan/robotic2/src/articubot_nuy/meshes/frontwheel.dae" scale="1 1 1"/>
+            </geometry>
+        </visual>
+        <collision>
+            <geometry>
+                <mesh filename="file:///home/preeyanan/robotic2/src/articubot_nuy/meshes/frontwheel.dae" scale="1 1 1"/>
             </geometry>
         </collision>
@@ -73,5 +73,5 @@
     </link>
     <gazebo reference="front_left_wheel">
-        <material>Gazebo/White</material>
+        <material>Gazebo/Black</material>
     </gazebo>
     <!-- === ล้อหน้า ขวา === -->
@@ -79,16 +79,16 @@
         <parent link="body"/>
         <child link="front_left_wheel"/>
-        <origin xyz="1 0.175 0" rpy="${pi/2} 0 0"/>
-        <axis xyz="-1 -1 0"/>
+        <origin xyz="-0.2007 -0.1481 0.0198" rpy="${pi/2} 0 0"/>
+        <axis xyz="1 0 0"/>
     </joint>
     <link name="front_right_wheel">
         <visual>
             <geometry>
-                <mesh filename="file:///home/preeyanan/miniproject/meshes/frontwheel.dae" scale="1 1 1"/>
-            </geometry>
-        </visual>
-        <collision>
-            <geometry>
-                <mesh filename="file:///home/preeyanan/miniproject/meshes/frontwheel.dae" scale="1 1 1"/>
+                <mesh filename="file:///home/preeyanan/robotic2/src/articubot_nuy/meshes/frontwheel.dae" scale="1 1 1"/>
+            </geometry>
+        </visual>
+        <collision>
+            <geometry>
+                <mesh filename="file:///home/preeyanan/robotic2/src/articubot_nuy/meshes/frontwheel.dae" scale="1 1 1"/>
             </geometry>
         </collision>
@@ -98,5 +98,5 @@
     </link>
     <gazebo reference="front_right_wheel">
-        <material>Gazebo/White</material>
+        <material>Gazebo/Black</material>
     </gazebo>
     <!-- === ล้อหลัง ซ้าย === -->
@@ -104,5 +104,5 @@
         <parent link="body"/>
         <child link="back_left_wheel"/>
-        <origin xyz="-0.5 1 0" rpy="${pi/2} 0 0"/>
+        <origin xyz="0.1925 0.1518 0.05" rpy="${pi/2} 0 0"/>
         <axis xyz="1 0 0"/>
     </joint>
@@ -110,10 +110,10 @@
         <visual>
             <geometry>
-                <mesh filename="file:///home/preeyanan/miniproject/meshes/backwheel.dae" scale="1 1 1"/>
-            </geometry>
-        </visual>
-        <collision>
-            <geometry>
-                <mesh filename="file:///home/preeyanan/miniproject/meshes/backwheel.dae" scale="1 1 1"/>
+                <mesh filename="file:///home/preeyanan/robotic2/src/articubot_nuy/meshes/backwheel.dae" scale="1 1 1"/>
+            </geometry>
+        </visual>
+        <collision>
+            <geometry>
+                <mesh filename="file:///home/preeyanan/robotic2/src/articubot_nuy/meshes/backwheel.dae" scale="1 1 1"/>
             </geometry>
         </collision>
@@ -123,5 +123,5 @@
     </link>
     <gazebo reference="back_left_wheel">
-        <material>Gazebo/White</material>
+        <material>Gazebo/Black</material>
     </gazebo>
     <!-- === ล้อหลัง ขวา === -->
@@ -129,5 +129,5 @@
         <parent link="body"/>
         <child link="back_right_wheel"/>
-        <origin xyz="-1 1 0" rpy="${pi/2} 0 0"/>
+        <origin xyz="-0.2017 0.1518 0.05" rpy="${pi/2} 0 0"/>
         <axis xyz="1 0 0"/>
     </joint>
@@ -135,10 +135,10 @@
         <visual>
             <geometry>
-                <mesh filename="file:///home/preeyanan/miniproject/meshes/backwheel.dae" scale="1 1 1"/>
-            </geometry>
-        </visual>
-        <collision>
-            <geometry>
-                <mesh filename="file:///home/preeyanan/miniproject/meshes/backwheel.dae" scale="1 1 1"/>
+                <mesh filename="file:///home/preeyanan/robotic2/src/articubot_nuy/meshes/backwheel.dae" scale="1 1 1"/>
+            </geometry>
+        </visual>
+        <collision>
+            <geometry>
+                <mesh filename="file:///home/preeyanan/robotic2/src/articubot_nuy/meshes/backwheel.dae" scale="1 1 1"/>
             </geometry>
         </collision>
@@ -148,5 +148,5 @@
     </link>
     <gazebo reference="back_right_wheel">
-        <material>Gazebo/White</material>
+        <material>Gazebo/Black</material>
     </gazebo>
     <!-- === LR L === -->
@@ -154,17 +154,17 @@
         <parent link="body"/>
         <child link="LR_L"/>
-        <origin xyz="0 1 0" rpy="0 0 0"/>
-        <axis xyz="1 0 0"/>
-        <limit lower="-1" upper="1" effort="1" velocity="1"/>
+        <origin xyz="0.066 -0.296 0.095" rpy="0 0 0"/>
+        <axis xyz="1 0 0"/>
+        <limit lower="0" upper="0.5" effort="1" velocity="1"/>
     </joint>
     <link name="LR_L">
         <visual>
             <geometry>
-                <mesh filename="file:///home/preeyanan/miniproject/meshes/LR.dae" scale="1 1 1"/>
-            </geometry>
-        </visual>
-        <collision>
-            <geometry>
-                <mesh filename="file:///home/preeyanan/miniproject/meshes/LR.dae" scale="1 1 1"/>
+                <mesh filename="file:///home/preeyanan/robotic2/src/articubot_nuy/meshes/LR.dae" scale="1 1 1"/>
+            </geometry>
+        </visual>
+        <collision>
+            <geometry>
+                <mesh filename="file:///home/preeyanan/robotic2/src/articubot_nuy/meshes/LR.dae" scale="1 1 1"/>
             </geometry>
         </collision>
@@ -182,15 +182,15 @@
         <origin xyz="-0.066 -0.296 0.095" rpy="0 0 0"/>
         <axis xyz="1 0 0"/>
-        <limit lower="-1" upper="1" effort="1" velocity="1"/>
+        <limit lower="-0.5" upper="0" effort="1" velocity="1"/>
     </joint>
     <link name="LR_R">
         <visual>
             <geometry>
-                <mesh filename="file:///home/preeyanan/miniproject/meshes/LR.dae" scale="1 1 1"/>
-            </geometry>
-        </visual>
-        <collision>
-            <geometry>
-                <mesh filename="file:///home/preeyanan/miniproject/meshes/LR.dae" scale="1 1 1"/>
+                <mesh filename="file:///home/preeyanan/robotic2/src/articubot_nuy/meshes/LR.dae" scale="1 1 1"/>
+            </geometry>
+        </visual>
+        <collision>
+            <geometry>
+                <mesh filename="file:///home/preeyanan/robotic2/src/articubot_nuy/meshes/LR.dae" scale="1 1 1"/>
             </geometry>
         </collision>
@@ -206,5 +206,5 @@
         <parent link="LR_L"/>
         <child link="UD_L"/>
-        <origin xyz="0 1.5 0" rpy="0 0 0"/>
+        <origin xyz="0 -0.03 0" rpy="0 0 0"/>
         <axis xyz="0 0 1"/>
         <limit lower="-1" upper="1" effort="1" velocity="1"/>
@@ -213,10 +213,10 @@
         <visual>
             <geometry>
-                <mesh filename="file:///home/preeyanan/miniproject/meshes/UDL.dae" scale="1 1 1"/>
-            </geometry>
-        </visual>
-        <collision>
-            <geometry>
-                <mesh filename="file:///home/preeyanan/miniproject/meshes/UDL.dae" scale="1 1 1"/>
+                <mesh filename="file:///home/preeyanan/robotic2/src/articubot_nuy/meshes/UDL.dae" scale="1 1 1"/>
+            </geometry>
+        </visual>
+        <collision>
+            <geometry>
+                <mesh filename="file:///home/preeyanan/robotic2/src/articubot_nuy/meshes/UDL.dae" scale="1 1 1"/>
             </geometry>
         </collision>
@@ -232,5 +232,5 @@
         <parent link="LR_R"/>
         <child link="UD_R"/>
-        <origin xyz="0 1 0" rpy="0 0 0"/>
+        <origin xyz="0 -0.03 0" rpy="0 0 0"/>
         <axis xyz="0 0 1"/>
         <limit lower="-1" upper="1" effort="1" velocity="1"/>
@@ -239,10 +239,10 @@
         <visual>
             <geometry>
-                <mesh filename="file:///home/preeyanan/miniproject/meshes/UDR.dae" scale="1 1 1"/>
-            </geometry>
-        </visual>
-        <collision>
-            <geometry>
-                <mesh filename="file:///home/preeyanan/miniproject/meshes/UDR.dae" scale="1 1 1"/>
+                <mesh filename="file:///home/preeyanan/robotic2/src/articubot_nuy/meshes/UDR.dae" scale="1 1 1"/>
+            </geometry>
+        </visual>
+        <collision>
+            <geometry>
+                <mesh filename="file:///home/preeyanan/robotic2/src/articubot_nuy/meshes/UDR.dae" scale="1 1 1"/>
             </geometry>
         </collision>
