Commit message: Update robot_core.xacro

File: robot_core.xacro (robot description, xacro)
@@ -54,5 +54,5 @@
         <parent link="body"/>
         <child link="front_right_wheel"/>
-        <origin xyz="0.193 -0.1481 0.0198" rpy="${pi/2} 0 0"/>
+        <origin xyz="0.193 -0.1481 0.0198" rpy="0 0 0"/>
         <axis xyz="1 0 0"/>
     </joint>
@@ -79,5 +79,5 @@
         <parent link="body"/>
         <child link="front_left_wheel"/>
-        <origin xyz="-0.2007 -0.1481 0.0198" rpy="${pi/2} 0 0"/>
+        <origin xyz="-0.2007 -0.1481 0.0198" rpy="0 0 0"/>
         <axis xyz="1 0 0"/>
     </joint>
@@ -104,5 +104,5 @@
         <parent link="body"/>
         <child link="back_left_wheel"/>
-        <origin xyz="0.1925 0.1518 0.05" rpy="${pi/2} 0 0"/>
+        <origin xyz="0.1925 0.1518 0.05" rpy="0 0 0"/>
         <axis xyz="1 0 0"/>
     </joint>
@@ -129,5 +129,5 @@
         <parent link="body"/>
         <child link="back_right_wheel"/>
-        <origin xyz="-0.2017 0.1518 0.05" rpy="${pi/2} 0 0"/>
+        <origin xyz="-0.2017 0.1518 0.05" rpy="0 0 0"/>
         <axis xyz="1 0 0"/>
     </joint>
@@ -154,7 +154,7 @@
         <parent link="body"/>
         <child link="LR_L"/>
-        <origin xyz="0.066 -0.296 0.095" rpy="0 0 0"/>
-        <axis xyz="1 0 0"/>
-        <limit lower="0" upper="0.5" effort="1" velocity="1"/>
+        <origin xyz="0.14 -0.296 0.095" rpy="0 0 0"/>
+        <axis xyz="1 0 0"/>
+        <limit lower="0" upper="0.1" effort="1" velocity="1"/>
     </joint>
     <link name="LR_L">
@@ -180,7 +180,7 @@
         <parent link="body"/>
         <child link="LR_R"/>
-        <origin xyz="-0.066 -0.296 0.095" rpy="0 0 0"/>
-        <axis xyz="1 0 0"/>
-        <limit lower="-0.5" upper="0" effort="1" velocity="1"/>
+        <origin xyz="-0.138 -0.296 0.095" rpy="0 0 0"/>
+        <axis xyz="1 0 0"/>
+        <limit lower="0" upper="0.02" effort="1" velocity="-1"/>
     </joint>
     <link name="LR_R">
@@ -208,5 +208,5 @@
         <origin xyz="0 -0.03 0" rpy="0 0 0"/>
         <axis xyz="0 0 1"/>
-        <limit lower="-1" upper="1" effort="1" velocity="1"/>
+        <limit lower="-0.05" upper="0.05" effort="1" velocity="1"/>
     </joint>
     <link name="UD_L">
@@ -234,5 +234,5 @@
         <origin xyz="0 -0.03 0" rpy="0 0 0"/>
         <axis xyz="0 0 1"/>
-        <limit lower="-1" upper="1" effort="1" velocity="1"/>
+        <limit lower="-0.05" upper="0.05" effort="1" velocity="1"/>
     </joint>
     <link name="UD_R">

Commit message: Update robot_core.xacro

File: robot_core.xacro (robot description, xacro)
@@ -154,7 +154,7 @@
         <parent link="body"/>
         <child link="LR_L"/>
-        <origin xyz="0.14 -0.296 0.095" rpy="0 0 0"/>
-        <axis xyz="1 0 0"/>
-        <limit lower="0" upper="0.1" effort="1" velocity="1"/>
+        <origin xyz="0.142 -0.296 0.095" rpy="0 0 0"/>
+        <axis xyz="1 0 0"/>
+        <limit lower="-0.125" upper="0" effort="1" velocity="-1"/>
     </joint>
     <link name="LR_L">
@@ -180,7 +180,7 @@
         <parent link="body"/>
         <child link="LR_R"/>
-        <origin xyz="-0.138 -0.296 0.095" rpy="0 0 0"/>
-        <axis xyz="1 0 0"/>
-        <limit lower="0" upper="0.02" effort="1" velocity="-1"/>
+        <origin xyz="-0.139 -0.296 0.095" rpy="0 0 0"/>
+        <axis xyz="1 0 0"/>
+        <limit lower="0" upper="0.125" effort="1" velocity="1"/>
     </joint>
     <link name="LR_R">

Commit message: Update robot_core.xacro

File: robot_core.xacro (robot description, xacro)
@@ -208,5 +208,5 @@
         <origin xyz="0 -0.03 0" rpy="0 0 0"/>
         <axis xyz="0 0 1"/>
-        <limit lower="-0.05" upper="0.05" effort="1" velocity="1"/>
+        <limit lower="-0.085" upper="0.085" effort="1" velocity="-1"/>
     </joint>
     <link name="UD_L">
@@ -234,5 +234,5 @@
         <origin xyz="0 -0.03 0" rpy="0 0 0"/>
         <axis xyz="0 0 1"/>
-        <limit lower="-0.05" upper="0.05" effort="1" velocity="1"/>
+        <limit lower="-0.085" upper="0.085" effort="1" velocity="-1"/>
     </joint>
     <link name="UD_R">

Commit message: Update robot_core.xacro

File: robot_core.xacro (robot description, xacro)
@@ -154,5 +154,5 @@
         <parent link="body"/>
         <child link="LR_L"/>
-        <origin xyz="0.142 -0.296 0.095" rpy="0 0 0"/>
+        <origin xyz="0.1425 -0.296 0.095" rpy="0 0 0"/>
         <axis xyz="1 0 0"/>
         <limit lower="-0.125" upper="0" effort="1" velocity="-1"/>
